File: PCB/keyboard.kicad_sch (KiCad schematic)
At the start: 139 parts, among them SW1 SW_Push, SW10 SW_Push, SW11 SW_Push, SW12 SW_Push, SW13 SW_Push, SW14 SW_Push, SW15 SW_Push, SW16 SW_Push, SW17 SW_Push, SW18 SW_Push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

Commit message: Added PCB
Connections:
- net GND: now also U1.13 (GND), U1.18 (GND), U1.23 (GND), U1.28 (GND), U1.3 (GND), U1.8 (GND)
- no-connect marks 16 -> 10
Other:
- moved on the sheet: U1
