File: PCB/keyboard.kicad_pcb (KiCad board)
At the start: 2 copper layers, 290 x 122 mm, 123 parts, among them SW1 SW_Push, SW10 SW_Push, SW11 SW_Push, SW12 SW_Push, SW13 SW_Push, SW14 SW_Push, SW15 SW_Push, SW16 SW_Push, SW17 SW_Push, SW18 SW_Push, SW19 SW_Push, SW2 SW_Push, SW20 SW_Push, SW21 SW_Push, SW22 SW_Push, SW23 SW_Push, SW24 SW_Push, SW25 SW_Push, SW26 SW_Push, SW27 SW_Push, SW28 SW_Push, SW29 SW_Push, SW3 SW_Push, SW30 SW_Push, SW31 SW_Push, SW32 SW_Push, SW33 SW_Push, SW34 SW_Push, SW35 SW_Push, SW36 SW_Push, SW37 SW_Push, SW38 SW_Push, SW39 SW_Push, SW4 SW_Push, SW40 SW_Push, SW41 SW_Push, SW42 SW_Push, SW43 SW_Push, SW44 SW_Push, SW45 SW_Push, SW46 SW_Push, SW47 SW_Push, SW48 SW_Push, SW49 SW_Push, SW5 SW_Push, SW50 SW_Push, SW51 SW_Push, SW52 SW_Push, SW53 SW_Push, SW54 SW_Push, SW55 SW_Push, SW56 SW_Push, SW57 SW_Push, SW58 SW_Push, SW59 SW_Push, SW6 SW_Push, SW60 SW_Push, SW61 SW_Push, SW7 SW_Push, SW8 SW_Push, SW9 SW_Push, U1 Pico

Commit message: add PCB
Parts:
- added D62: 1N4148, Diode_THT:D_DO-35_SOD27_P7.62mm_Horizontal, B.Cu at (286.0, 96.8)
- added D63: 1N4148, Diode_THT:D_DO-35_SOD27_P7.62mm_Horizontal, B.Cu at (314.0, 96.6)
- added D64: SK6812MINI, LED_SMD:LED_SK6812MINI_PLCC4_3.5x3.5mm_P1.75mm, F.Cu at (124.2, 93.4)
- added D65: SK6812MINI, LED_SMD:LED_SK6812MINI_PLCC4_3.5x3.5mm_P1.75mm, F.Cu at (134.2, 93.4)
- added D66: SK6812MINI, LED_SMD:LED_SK6812MINI_PLCC4_3.5x3.5mm_P1.75mm, F.Cu at (144.2, 93.4)
- added D67: SK6812MINI, LED_SMD:LED_SK6812MINI_PLCC4_3.5x3.5mm_P1.75mm, F.Cu at (154.2, 93.4)
- added D68: SK6812MINI, LED_SMD:LED_SK6812MINI_PLCC4_3.5x3.5mm_P1.75mm, F.Cu at (164.2, 93.4)
- added D69: SK6812MINI, LED_SMD:LED_SK6812MINI_PLCC4_3.5x3.5mm_P1.75mm, F.Cu at (174.2, 93.4)
- added D70: SK6812MINI, LED_SMD:LED_SK6812MINI_PLCC4_3.5x3.5mm_P1.75mm, F.Cu at (184.2, 93.4)
- added D71: SK6812MINI, LED_SMD:LED_SK6812MINI_PLCC4_3.5x3.5mm_P1.75mm, F.Cu at (194.2, 93.4)
- added D72: SK6812MINI, LED_SMD:LED_SK6812MINI_PLCC4_3.5x3.5mm_P1.75mm, F.Cu at (204.2, 93.4)
- added D73: SK6812MINI, LED_SMD:LED_SK6812MINI_PLCC4_3.5x3.5mm_P1.75mm, F.Cu at (214.2, 93.4)
- added G***: LOGO, LOGO, F.Cu at (275.0, 92.0)
- added G***: LOGO, LOGO, F.Cu at (197.3, 192.9)
- added G***: LOGO, LOGO, F.Cu at (137.5, 192.6)
- added G***: LOGO, LOGO, F.Cu at (282.2, 132.9)
- added G***: LOGO, LOGO, F.Cu at (109.1, 90.3)
- added G***: LOGO, LOGO, F.Cu at (242.2, 166.5)
- added G***: LOGO, LOGO, B.Cu at (271.1, 170.6)
- added G***: LOGO, LOGO, B.Cu at (116.9, 136.4)
- added G***: LOGO, LOGO, F.Cu at (71.8, 131.2)
- added G***: LOGO, LOGO, F.Cu at (162.9, 150.5)
- added G***: LOGO, LOGO, F.Cu at (304.0, 92.5)
- added G***: LOGO, LOGO, F.Cu at (231.1, 91.8)
- added G***: LOGO, LOGO, F.Cu at (49.8, 179.4)
- added G***: LOGO, LOGO, F.Cu at (169.5, 89.2)
- added G***: LOGO, LOGO, F.Cu at (209.7, 120.3)
- added G***: LOGO, LOGO, F.Cu at (305.5, 178.3)
- added SW62: RotaryEncoder_Switch, Rotary_Encoder:RotaryEncoder_Alps_EC11E-Switch_Vertical_H20mm_CircularMountingHoles, F.Cu at (267.8, 89.5)
- added SW63: RotaryEncoder_Switch, Rotary_Encoder:RotaryEncoder_Alps_EC11E-Switch_Vertical_H20mm_CircularMountingHoles, F.Cu at (296.8, 90.0)
- D1, D10, D11, D12, D13, D14, D15, D16, D17, D18, D19, D2, D20, D21, D22, D23, D24, D25, D26, D27, D28, D29, D3, D30, D31, D32, D33, D34, D35, D36, D37, D38, D39, D4, D40, D41, D42, D43, D44, D45, D46, D47, D48, D49, D5, D50, D51, D52, D53, D54, D55, D56, D57, D58, D59, D6, D60, D61, D7, D8, D9: moved to B.Cu
- moved D54 296.8 mm to (35.0, 195.0), turned to 90 degrees
- moved D42 275.5 mm to (35.0, 175.8), turned to 90 degrees
- moved D55 275.1 mm to (59.0, 195.0), turned to 90 degrees
- moved D29 257.2 mm to (35.0, 157.8), turned to 90 degrees
- moved D56 254.3 mm to (82.0, 194.6), turned to 90 degrees
- moved D15 240.1 mm to (35.0, 137.8), turned to 90 degrees
- moved D43 238.3 mm to (77.0, 175.6), turned to 90 degrees
- moved D57 233.5 mm to (106.0, 194.6), turned to 90 degrees
- moved D30 226.4 mm to (68.0, 156.8), turned to 90 degrees
- moved D1 223.7 mm to (35.0, 118.8), turned to 90 degrees
- moved D44 220.2 mm to (97.0, 175.8), turned to 90 degrees
- moved D16 213.6 mm to (63.0, 137.8), turned to 90 degrees
- moved D31 208.5 mm to (87.0, 156.8), turned to 90 degrees
- moved D2 204.9 mm to (54.0, 118.6), turned to 90 degrees
- moved D45 203.2 mm to (116.0, 175.8), turned to 90 degrees
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Connections:
- U1 pad 25: unconnected-(U1-GPIO19-Pad25) -> re1
- U1 pad 26: unconnected-(U1-GPIO20-Pad26) -> re2
- U1 pad 27: unconnected-(U1-GPIO21-Pad27) -> re3
- U1 pad 29: unconnected-(U1-GPIO22-Pad29) -> re4
- U1 pad 31: unconnected-(U1-GPIO26_ADC0-Pad31) -> rgb1
- U1 pad 32: unconnected-(U1-GPIO27_ADC1-Pad32) -> rgb2
- U1 pad 38: unconnected-(U1-GND-Pad38) -> GND
- U1 pad 40: unconnected-(U1-VBUS-Pad40) -> +5V
Routing:
- net row4: track 0.00 -> 463.8 mm, vias 0 -> 3
- net row3: track 0.00 -> 451.9 mm, vias 0 -> 1
- net row5: track 0.00 -> 438.4 mm, vias 0 -> 5
- net row2: track 0.00 -> 347.3 mm
- net col8: track 0.00 -> 329.9 mm
- net col7: track 0.00 -> 311.8 mm
- net col14: track 0.00 -> 307.0 mm
- net GND: track 0.00 -> 290.1 mm, vias 0 -> 1
- net col6: track 0.00 -> 287.9 mm
- net col12: track 0.00 -> 287.1 mm
- net col13: track 0.00 -> 273.5 mm
- net row1: track 0.00 -> 270.1 mm
- net col5: track 0.00 -> 265.7 mm
- net col11: track 0.00 -> 253.5 mm
- net re4: track 0.00 -> 240.1 mm
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Other:
- board size 290 x 122 mm -> 290.8 x 123.2 mm

Commit message: journal: day-3
Parts:
- removed D73: SK6812MINI, LED_SMD:LED_SK6812MINI_PLCC4_3.5x3.5mm_P1.75mm
- added R1: 330Ω, Resistor_THT:R_Axial_DIN0309_L9.0mm_D3.2mm_P20.32mm_Horizontal, B.Cu at (121.0, 86.8)
- added R2: 330Ω, Resistor_THT:R_Axial_DIN0309_L9.0mm_D3.2mm_P20.32mm_Horizontal, B.Cu at (121.0, 93.2)
- added R3: 330Ω, Resistor_THT:R_Axial_DIN0309_L9.0mm_D3.2mm_P20.32mm_Horizontal, B.Cu at (121.2, 99.2)
- D64, D65, D66, D67, D68, D69, D70, D71, D72: value SK6812MINI -> LED_Small; footprint LED_SMD:LED_SK6812MINI_PLCC4_3.5x3.5mm_P1.75mm -> LED_THT:LED_D5.0mm
- moved D64 69.2 mm to (193.5, 95.0)
- moved D70 47.3 mm to (137.0, 94.0)
- moved D67 47.1 mm to (201.0, 87.8), turned to 90 degrees
- moved D72 34.6 mm to (170.5, 86.0)
- moved D65 15.3 mm to (148.0, 86.5)
- moved D69 9.77 mm to (184.0, 94.0), turned to -90 degrees
- moved D71 9.26 mm to (202.0, 98.5)
- moved G*** 6.13 mm to (237.1, 91.2)
- moved D66 6.01 mm to (150.2, 94.0)
- moved G*** 4.20 mm to (105.1, 91.7)
- moved D68 0.80 mm to (163.5, 93.5)
Connections:
- D64 pad 1: unconnected-(D64-DOUT-Pad1) -> Net-(D64-K)
- D64 pad 2: GND -> red_anode
- D65 pad 1: unconnected-(D65-DOUT-Pad1) -> Net-(D64-K)
- D65 pad 2: GND -> red_anode
- D66 pad 1: unconnected-(D66-DOUT-Pad1) -> Net-(D64-K)
- D66 pad 2: GND -> red_anode
- D67 pad 1: unconnected-(D67-DOUT-Pad1) -> Net-(D67-K)
- D67 pad 2: GND -> blue_anode
- D68 pad 1: unconnected-(D68-DOUT-Pad1) -> Net-(D67-K)
- D68 pad 2: GND -> blue_anode
- D69 pad 1: unconnected-(D69-DOUT-Pad1) -> Net-(D67-K)
- D69 pad 2: GND -> blue_anode
- D70 pad 1: unconnected-(D70-DOUT-Pad1) -> Net-(D70-K)
- D70 pad 2: GND -> green_anode
- D71 pad 1: unconnected-(D71-DOUT-Pad1) -> Net-(D70-K)
- D71 pad 2: GND -> green_anode
- D72 pad 1: unconnected-(D72-DOUT-Pad1) -> Net-(D70-K)
- D72 pad 2: GND -> green_anode
- U1 pad 31: rgb1 -> green_anode
- U1 pad 32: rgb2 -> red_anode
- U1 pad 34: unconnected-(U1-GPIO28_ADC2-Pad34) -> blue_anode
- U1 pad 40: +5V -> unconnected-(U1-VBUS-Pad40)
Routing:
- net +5V: track 196.4 -> 0.00 mm, vias 2 -> 0
- net green_anode: track 0.00 -> 174.5 mm, vias 0 -> 2
- net blue_anode: track 0.00 -> 164.9 mm, vias 0 -> 1
- net red_anode: track 0.00 -> 164.5 mm, vias 0 -> 2
- net rgb2: track 135.7 -> 0.00 mm, vias 5 -> 0
- net Net-(D70-K): track 0.00 -> 102.4 mm
- net Net-(D67-K): track 0.00 -> 100.0 mm
- net Net-(D64-K): track 0.00 -> 98.1 mm
- net rgb1: track 74.6 -> 0.00 mm, vias 1 -> 0
- net GND: track 290.1 -> 325.2 mm, vias 1 -> 4
Other:
- board size 290.8 x 123.2 mm -> 290.9 x 123.4 mm

Commit message: Added PCB
Parts:
- moved D70 113.2 mm to (249.5, 106.2)
- moved D65 43.7 mm to (187.0, 106.2)
- moved D67 40.4 mm to (237.0, 106.2), turned to 0 degrees
- moved D68 38.2 mm to (199.5, 106.2)
- moved G*** 34.1 mm to (306.0, 106.2)
- moved SW62 34.1 mm to (298.8, 103.7)
- moved D62 33.4 mm to (316.5, 110.5)
- moved D64 32.9 mm to (224.5, 106.2)
- moved G*** 32.5 mm to (271.7, 180.2)
- moved SW38 32.5 mm to (262.1, 161.1)
- moved SW51 32.5 mm to (271.7, 180.2)
- moved G*** 32.5 mm to (134.6, 105.4)
- moved SW32 32.5 mm to (147.8, 161.1)
- moved D1 32.5 mm to (64.5, 132.5)
- moved D10 32.5 mm to (235.5, 132.3)
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Connections:
- U1 pad 13: unconnected-(U1-GND-Pad13)_1 -> GND
- U1 pad 18: unconnected-(U1-GND-Pad18) -> GND
- U1 pad 23: unconnected-(U1-GND-Pad23)_1 -> GND
- U1 pad 28: unconnected-(U1-GND-Pad28) -> GND
- U1 pad 3: unconnected-(U1-GND-Pad3)_1 -> GND
- U1 pad 8: unconnected-(U1-GND-Pad8)_1 -> GND
Routing:
- net GND: track 325.2 -> 404.7 mm, vias 4 -> 6
- net green_anode: track 174.5 -> 197.7 mm
- net Net-(D70-K): track 102.4 -> 122.4 mm
- net blue_anode: track 164.9 -> 173.3 mm, vias 1 -> 2
- net red_anode: track 164.5 -> 156.0 mm, vias 2 -> 4
- net Net-(D67-K): track 100.0 -> 106.6 mm, vias 0 -> 1
- net Net-(D64-K): track 98.1 -> 96.3 mm, vias 0 -> 2
- net re2: track 203.9 -> 205.6 mm
- net re1: track 204.5 -> 206.2 mm
- net col2: track 140.7 -> 140.1 mm
